File: pnp/pcb/mobo/dual_motors.kicad_sch (KiCad schematic)
At the start: 9 parts, among them M5 MOTOR1, M6 MOTOR2

Commit message: Add manufacturer and partnumber field
Parts:
- C21: Manufacturer (none) -> s
Changed lines of the file:
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@@
+      (effects (font (size 1.27 1.27)) hide)
+    )
+    (property "Manufacturer" "s" (id 8) (at 165.735 48.26 0)
       (effects (font (size 1.27 1.27)) hide)
     )
