File: pnp/pcb/mobo/dual_motors.kicad_sch (KiCad schematic)
At the start: 9 parts, among them M5 MOTOR1, M6 MOTOR2

Commit message: Test version replacement in title block
Other:
- title: (none) -> Index Mobo
Changed lines of the file:
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@@
 (kicad_sch (version 20211123) (generator eeschema)
   (paper "A4")
+  (title_block
+    (title "Index Mobo")
+    (date "2021-02-19")
+    (rev "${version}")
+  )
   (junction (at 149.86 82.55) (diameter 0) (color 0 0 0 0)
   )
