File: pnp/pcb/mobo/misc_input.kicad_sch (KiCad schematic)
At the start: 26 parts, among them J2 X_LIMIT, J3 Y_LIMIT, J4 Z_LIMIT, J5 L_LIMIT, J6 R_LIMIT, J7 A_LIMIT, U2 TL072, U3 XGZP101SB1, U4 2SMPP-03, U5 XGZP101SB1, U6 2SMPP-03, U7 INA128, U8 INA128, U9 MCP3426-xMS

Commit message: Add manufacturer and partnumber field
Parts:
- FB2: Manufacturer (none) -> a; Partnumber (none) -> a
- J7: Partnumber (none) -> f
Changed lines of the file:
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@@
+      (effects (font (size 1.27 1.27)) hide)
+    )
+    (property "Manufacturer" "a" (id 6) (at 201.93 69.85 0)
+      (effects (font (size 1.27 1.27)) hide)
+    )
+    (property "Partnumber" "a" (id 7) (at 201.93 69.85 0)
       (effects (font (size 1.27 1.27)) hide)
     )
@@
       (effects (font (size 1.27 1.27)) hide)
     )
+    (property "Partnumber" "f" (id 7) (at 65.405 132.08 0)
+      (effects (font (size 1.27 1.27)) hide)
+    )
