File: pnp/pcb/mobo/mobo.kicad_sch (KiCad schematic)
At the start: 38 parts, among them J1 SWD Header, SW1 SW_Push, SW2 SW_Push, U1 STM32F407VETx, Y1 8MHz

Commit message: Add manufacturer and partnumber field
Parts:
- C1, C14, C3, C6, C7: Partnumber (none) -> a
- FB1: Manufacturer (none) -> a; Partnumber (none) -> a
Changed lines of the file:
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@@
+      (effects (font (size 1.27 1.27)) hide)
+    )
+    (property "Partnumber" "a" (id 8) (at 36.83 66.04 0)
       (effects (font (size 1.27 1.27)) hide)
     )
@@
     )
     (property "Mouser" "963-UMK212ABJ225KG-T" (id 7) (at 43.18 68.58 0)
+      (effects (font (size 1.27 1.27)) hide)
+    )
+    (property "Partnumber" "a" (id 8) (at 43.18 68.58 0)
       (effects (font (size 1.27 1.27)) hide)
     )
@@
       (effects (font (size 1.27 1.27)) hide)
     )
+    (property "Partnumber" "a" (id 8) (at 27.305 26.035 0)
+      (effects (font (size 1.27 1.27)) hide)
+    )
     (pin "1")
     (pin "2")
@@
       (effects (font (size 1.27 1.27)) hide)
     )
+    (property "Partnumber" "a" (id 8) (at 19.05 26.035 0)
+      (effects (font (size 1.27 1.27)) hide)
+    )
     (pin "1")
     (pin "2")
@@
     )
     (property "Mouser" "963-UMK212ABJ225KG-T" (id 7) (at 123.19 26.035 0)
+      (effects (font (size 1.27 1.27)) hide)
+    )
+    (property "Partnumber" "a" (id 8) (at 123.19 26.035 0)
       (effects (font (size 1.27 1.27)) hide)
     )
@@
       (effects (font (size 1.27 1.27)) hide)
     )
+    (property "Manufacturer" "a" (id 6) (at 106.68 23.495 0)
+      (effects (font (size 1.27 1.27)) hide)
+    )
+    (property "Partnumber" "a" (id 7) (at 106.68 23.495 0)
+      (effects (font (size 1.27 1.27)) hide)
+    )
