File: pnp/pcb/mobo/motor.kicad_sch (KiCad schematic)
At the start: 8 parts, among them M4 Stepper_Motor

Commit message: Add manufacturer and partnumber field
Parts:
- C20: Manufacturer (none) -> s
Changed lines of the file:
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@@
+      (effects (font (size 1.27 1.27)) hide)
+    )
+    (property "Manufacturer" "s" (id 8) (at 153.67 59.055 0)
       (effects (font (size 1.27 1.27)) hide)
     )
