File: pnp/pcb/mobo/motor.kicad_sch (KiCad schematic)
At the start: 8 parts, among them M4 Stepper_Motor

Commit message: Test version replacement in title block
Other:
- title: Motor -> Index Mobo
Changed lines of the file:
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@@
   (paper "A4")
   (title_block
-    (title "Motor")
+    (title "Index Mobo")
     (date "2021-02-19")
-    (rev "003")
+    (rev "${version}")
   )
   (junction (at 117.475 115.57) (diameter 0) (color 0 0 0 0)
