File: pnp/pcb/mobo/power.kicad_sch (KiCad schematic)
At the start: 28 parts, among them J12 Power, U11 FDS4435BZ, U12 TPS54331, U13 AP1117-33

Commit message: Add manufacturer and partnumber field
Parts:
- C27: Manufacturer (none) -> s
Changed lines of the file:
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@@
+      (effects (font (size 1.27 1.27)) hide)
+    )
+    (property "Manufacturer" "s" (id 8) (at 67.31 97.155 0)
       (effects (font (size 1.27 1.27)) hide)
     )
