File: pnp/pcb/mobo/power.kicad_sch (KiCad schematic)
At the start: 28 parts, among them J12 Power, U11 FDS4435BZ, U12 TPS54331, U13 AP1117-33

Commit message: Test version replacement in title block
Other:
- title: Power -> Index Mobo
Changed lines of the file:
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@@
   (paper "A4")
   (title_block
-    (title "Power")
+    (title "Index Mobo")
     (date "2021-02-19")
-    (rev "003")
+    (rev "${version}")
   )
   (junction (at 45.72 98.425) (diameter 0) (color 0 0 0 0)

Commit message: Clean up, working
Parts:
- removed C27: 100u, Capacitor_SMD:CP_Elec_6.3x7.7, symbol Device:CP
- removed C28, C29: 10n, Capacitor_SMD:C_0805_2012Metric, symbol Device:C
- removed C30: 2.2n, Capacitor_SMD:C_0805_2012Metric, symbol Device:C
- removed C31: 22p, Capacitor_SMD:C_0805_2012Metric, symbol Device:C
- removed C32: 100n, Capacitor_SMD:C_0805_2012Metric, symbol Device:C_Small
- removed C33, C34, C35: 22u, Capacitor_SMD:C_0805_2012Metric, symbol Device:C
- removed C36: 10u, Capacitor_SMD:C_0805_2012Metric, symbol Device:C
- removed D2: Yellow, LED_SMD:LED_0805_2012Metric, symbol Device:LED
- removed D3: SS34, Diode_SMD:D_SMA, symbol Device:D_Schottky
- removed D4, D5: CUS10S30, Diode_SMD:D_SOD-323, symbol Device:D_Schottky
- removed J12: Power, TerminalBlock_Phoenix:TerminalBlock_Phoenix_MKDS-1,5-2_1x02_P5.00mm_Horizontal, symbol Connector:Screw_Terminal_01x02
- removed JP26: EN_VBUS, Jumper:SolderJumper-2_P1.3mm_Bridged_RoundedPad1.0x1.5mm, symbol Jumper:SolderJumper_2_Bridged
- removed L1: 12u, Inductor_SMD:L_Coilcraft_XAL60xx_6.36x6.56mm, symbol pspice:INDUCTOR
- removed R24, R26: 10k, Resistor_SMD:R_0805_2012Metric, symbol Device:R_Small
- removed R25: 12.1k, Resistor_SMD:R_0805_2012Metric, symbol Device:R
- removed R27: 1.91k, Resistor_SMD:R_0805_2012Metric, symbol Device:R_Small
- removed TP10: 3V3_TestPoint, TestPoint:TestPoint_Pad_D2.0mm, symbol Connector:TestPoint
- removed TP7: GND_TestPoint, TestPoint:TestPoint_Pad_D2.0mm, symbol Connector:TestPoint
- removed TP8: VDC_TestPoint, TestPoint:TestPoint_Pad_D2.0mm, symbol Connector:TestPoint
- removed TP9: 5V_TestPoint, TestPoint:TestPoint_Pad_D2.0mm, symbol Connector:TestPoint
- removed U11: FDS4435BZ, Package_SO:SO-8_3.9x4.9mm_P1.27mm, symbol index:FDS4435BZ
- removed U12: TPS54331, Package_SO:SOIC-8_3.9x4.9mm_P1.27mm, symbol index:TPS54331
- removed U13: AP1117-33, Package_TO_SOT_SMD:SOT-223-3_TabPin2, symbol Regulator_Linear:AP1117-33
- added C1: 1uF 35V, Capacitor_SMD:C_0805_2012Metric, symbol Device:C_Small
- added C16: 220uF 35V, Capacitor_SMD:CP_Elec_10x10, symbol Device:C_Polarized_Small
- added C17: 100nF 50V, Capacitor_SMD:C_0603_1608Metric, symbol Device:C_Small
- added C2: 22uF 35V, Capacitor_SMD:CP_Elec_5x5.8, symbol Device:C_Polarized_Small
- added D4, D5: Green, LED_SMD:LED_0805_2012Metric, symbol Device:LED_Small
- added D6: 1.5SMC33CA-E3/57T, Diode_SMD:D_SMC, symbol Device:D_Small
- added J25: Molex MegaFit 01x02, Connector_Molex:Molex_Mega-Fit_76825-0002_2x01_P5.70mm_Horizontal, symbol Connector_Generic:Conn_01x02
- added R18: 1k, Resistor_SMD:R_0603_1608Metric, symbol Device:R_Small
- added R19: 4k7, Resistor_SMD:R_0603_1608Metric, symbol Device:R_Small
- added U7: LM2931-5.0_SO8, Package_SO:SOIC-8_3.9x4.9mm_P1.27mm, symbol Regulator_Linear:LM2931-5.0_SO8
Connections:
- net +5V: now also C2.1, D4.2 (A), U7.1 (OUT)
- net GND: now also C1.2, C16.2, C17.2, C2.2, D6.2 (A), J25.1 (Pin_1), R18.2, R19.2, U7.2 (GND), U7.3 (GND), U7.6 (GND), U7.7 (GND)
- new net: D4.1 (K), R18.1
- new net: D5.1 (K), R19.1
- new net +24V: C1.1, C16.1, C17.1, D5.2 (A), D6.1 (K), J25.2 (Pin_2), U7.8 (IN)
- no-connect marks 1 -> 0
Other:
- note added: "24V power input"
- note added: "5V regulator"
- note added: "Power indication leds"
- company: (none) -> 3devo
- title: Index Mobo -> GD BLDC blower driver
