File: pnp/pcb/mobo/usb.kicad_sch (KiCad schematic)
At the start: 15 parts, among them J10 AUX USB, J11 Top Camera, J8 Host, J9 Bottom Camera, U10 FE1.1, Y2 12MHz

Commit message: Add manufacturer and partnumber field
Parts:
- J11: Manufacturer (none) -> a
Changed lines of the file:
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@@
+      (effects (font (size 1.27 1.27)) hide)
+    )
+    (property "Manufacturer" "a" (id 8) (at 208.28 89.535 0)
       (effects (font (size 1.27 1.27)) hide)
     )
