File: pnp/pcb/mobo/misc_output.kicad_sch (KiCad schematic)
At the start: 12 parts, among them J13 DOWNWARDS_LIGHT, J14 UPWARDS_LIGHT, J15 SERVO1, J16 SERVO2, J17 Feeders, J18 AUX1, J19 AUX2, J20 AUX3, J21 qwiic, U14 MAX3078E

Commit message: Add manufacturer and partnumber field
Parts:
- J17: Partnumber (none) -> f
Changed lines of the file:
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@@
+      (effects (font (size 1.27 1.27)) hide)
+    )
+    (property "Partnumber" "f" (id 6) (at 123.825 128.905 0)
       (effects (font (size 1.27 1.27)) hide)
     )

Commit message: Test version replacement in title block
Other:
- title: Output -> Index Mobo
Changed lines of the file:
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@@
   (paper "A4")
   (title_block
-    (title "Output")
+    (title "Index Mobo")
     (date "2021-02-19")
-    (rev "003")
+    (rev "${version}")
   )
   (junction (at 117.475 123.825) (diameter 0) (color 0 0 0 0)
