File: pnp/pcb/mobo/mosfet.kicad_sch (KiCad schematic)
At the start: 5 parts, among them J25 Mosfet, Q4 AO3400A

Commit message: Test version replacement in title block
Other:
- title: Mosfet -> Index Mobo
Changed lines of the file:
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@@
   (paper "A4")
   (title_block
-    (title "Mosfet")
+    (title "Index Mobo")
     (date "2021-02-19")
-    (rev "003")
+    (rev "${version}")
   )
   (junction (at 144.78 93.345) (diameter 0) (color 0 0 0 0)
