File: pnp/pcb/mobo/motor_control.kicad_sch (KiCad schematic)
At the start: 0 parts

Commit message: Test version replacement in title block
Other:
- title: Motors -> Index Mobo
Changed lines of the file:
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@@
   (paper "A4")
   (title_block
-    (title "Motors")
+    (title "Index Mobo")
     (date "2021-02-19")
-    (rev "003")
+    (rev "${version}")
   )
   (hierarchical_label "COPI" (shape input) (at 181.61 99.06 0)
