File: PCB/mobo/mobo.kicad_pcb (KiCad board)
At the start: 2 copper layers, 100 x 80 mm, 99 parts, among them J1 Conn_02x06, J10 TEST_1P, J11 TEST_1P, J12 TEST_1P, J13 TEST_1P, J14 TEST_1P, J15 TEST_1P, J16 TEST_1P, J17 TEST_1P, J18 TEST_1P, J19 TEST_1P, J2 CONN_01X01, J20 TEST_1P, J21 TEST_1P, J22 TEST_1P, J23 TEST_1P, J24 TEST_1P, J25 Conn_01x02, J26 TEST_1P, J27 TEST_1P, J28 CONN_01X01, J3 CONN_01X01, J4 TEST_1P, J5 Conn_01x08, J6 Conn_01x05_Female, J7 TEST_1P, J8 TEST_1P, J9 TEST_1P, U1 MAX14851, U2 MAX14851, U3 DRV8308, U4 CSD88537ND, U5 CSD88537ND, U6 CSD88537ND, U7 LM2931-5.0_SO8, X1 Logo

Commit message: Date/rev added correctly to kicad 6 files
Other:
- board text added: "${version}"
Changed lines of the file:
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@@
   (title_block
     (title "GD motor driver test")
-    (date "2019-03-11")
-    (rev "1.2")
+    (date "${date}")
+    (rev "${version}")
     (company "3devo")
   )
@@
     )
   )
-  (property "version" "1.2.3")
   (net 0 "")
   (net 1 "GND")
@@
     (effects (font (size 1 1) (thickness 0.25)))
   )
+  (gr_text "${version}" (at 98.85 177) (layer "F.SilkS")
+    (effects (font (size 1.5 1.5) (thickness 0.3)))
+  )
   (gr_text "+" (at 56.3 120.3) (layer "F.SilkS")
