File: PCB/mobo/Driver.kicad_sch (KiCad schematic)
At the start: 41 parts, among them J10 Testpoint, J11 Testpoint, J12 Testpoint, J13 Testpoint, J14 Testpoint, J15 Testpoint, J16 Testpoint, J17 Testpoint, J18 Testpoint, J19 Testpoint, J20 Testpoint, J21 Testpoint, J22 Testpoint, J23 Testpoint, J24 Testpoint, J26 Testpoint, J27 Testpoint, J28 Testpoint, J4 Testpoint, J7 Testpoint, J8 Testpoint, J9 Testpoint, U3 DRV8308

Commit message: Pretty stable naming and xlsx output
Parts:
- R10, R9: Config (none) -> -SR
Changed lines of the file:
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@@
+      (effects (font (size 1.27 1.27)) hide)
+    )
+    (property "Config" "-SR" (id 6) (at 198.12 139.7 0)
       (effects (font (size 1.27 1.27)) hide)
     )
@@
       (effects (font (size 1.27 1.27)) hide)
     )
+    (property "Config" "-SR" (id 6) (at 198.12 132.08 0)
+      (effects (font (size 1.27 1.27)) hide)
+    )
