File: PCB/mobo/Inputs.kicad_sch (KiCad schematic)
At the start: 32 parts, among them J1 Pinheader 02x06 shrouded, J2 Testpoint, J3 Testpoint, U1 MAX14851, U2 MAX14851

Commit message: Pretty stable naming and xlsx output
Parts:
- J1: Config (none) -> +SR
- R1, R12, R14, R15, R16, R2, R20, R21, R22, R23, R26, R27, R28, R29, R3, R31, R5: Config (none) -> -SR
- U1: Config (none) -> +GR
Changed lines of the file:
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@@
+      (effects (font (size 1.27 1.27)) hide)
+    )
+    (property "Config" "-SR" (id 6) (at 198.12 111.76 0)
       (effects (font (size 1.27 1.27)) hide)
     )
@@
     )
     (property "Partnumber" "CR0603-FX-1002GLF" (id 5) (at 127 132.08 0)
+      (effects (font (size 1.27 1.27)) hide)
+    )
+    (property "Config" "-SR" (id 6) (at 127 132.08 0)
       (effects (font (size 1.27 1.27)) hide)
     )
@@
       (effects (font (size 1.27 1.27)) hide)
     )
+    (property "Config" "+GR" (id 8) (at 175.26 67.31 0)
+      (effects (font (size 1.27 1.27)) hide)
+    )
     (pin "1")
     (pin "10")
@@
       (effects (font (size 1.27 1.27)) hide)
     )
+    (property "Config" "-SR" (id 6) (at 142.24 111.76 0)
+      (effects (font (size 1.27 1.27)) hide)
+    )
     (pin "1")
     (pin "2")
@@
     )
     (property "Partnumber" "CR0603-FX-1002GLF" (id 5) (at 237.49 119.38 0)
+      (effects (font (size 1.27 1.27)) hide)
+    )
+    (property "Config" "-SR" (id 6) (at 237.49 119.38 0)
       (effects (font (size 1.27 1.27)) hide)
     )
@@
       (effects (font (size 1.27 1.27)) hide)
     )
+    (property "Config" "-SR" (id 6) (at 134.62 78.74 0)
+      (effects (font (size 1.27 1.27)) hide)
+    )
     (pin "1")
     (pin "2")
@@
       (effects (font (size 1.27 1.27)) hide)
     )
+    (property "Config" "-SR" (id 6) (at 205.74 111.76 0)
+      (effects (font (size 1.27 1.27)) hide)
+    )
     (pin "1")
     (pin "2")
@@
       (effects (font (size 1.27 1.27)) hide)
     )
+    (property "Config" "-SR" (id 6) (at 157.48 132.08 0)
+      (effects (font (size 1.27 1.27)) hide)
+    )
     (pin "1")
     (pin "2")
@@
     )
     (property "Partnumber" "CR0603-FX-1002GLF" (id 5) (at 149.86 132.08 0)
+      (effects (font (size 1.27 1.27)) hide)
+    )
+    (property "Config" "-SR" (id 6) (at 149.86 132.08 0)
       (effects (font (size 1.27 1.27)) hide)
     )
@@
       (effects (font (size 1.27 1.27)) hide)
     )
+    (property "Config" "-SR" (id 6) (at 232.41 66.04 0)
+      (effects (font (size 1.27 1.27)) hide)
+    )
     (pin "1")
     (pin "2")
@@
     )
     (property "Partnumber" "CR0603-FX-1002GLF" (id 5) (at 147.32 78.74 0)
+      (effects (font (size 1.27 1.27)) hide)
+    )
+    (property "Config" "-SR" (id 6) (at 147.32 78.74 0)
       (effects (font (size 1.27 1.27)) hide)
     )
@@
       (effects (font (size 1.27 1.27)) hide)
     )
+    (property "Config" "-SR" (id 6) (at 213.36 111.76 0)
+      (effects (font (size 1.27 1.27)) hide)
+    )
     (pin "1")
     (pin "2")
@@
     )
     (property "Partnumber" "CR0603-FX-1002GLF" (id 5) (at 232.41 123.19 0)
+      (effects (font (size 1.27 1.27)) hide)
+    )
+    (property "Config" "-SR" (id 6) (at 232.41 123.19 0)
       (effects (font (size 1.27 1.27)) hide)
     )
@@
       (effects (font (size 1.27 1.27)) hide)
     )
+    (property "Config" "-SR" (id 6) (at 236.22 62.23 0)
+      (effects (font (size 1.27 1.27)) hide)
+    )
     (pin "1")
     (pin "2")
@@
     )
     (property "Partnumber" "CR0603-FX-1002GLF" (id 5) (at 205.74 57.15 0)
+      (effects (font (size 1.27 1.27)) hide)
+    )
+    (property "Config" "-SR" (id 6) (at 205.74 57.15 0)
       (effects (font (size 1.27 1.27)) hide)
     )
@@
     (property "Function" "MCU I/O" (id 7) (at 64.77 82.55 0))
     (property "Partnumber" "T821112A1S100CEU" (id 8) (at 63.5 91.44 0)
+      (effects (font (size 1.27 1.27)) hide)
+    )
+    (property "Config" "+SR" (id 9) (at 63.5 91.44 0)
       (effects (font (size 1.27 1.27)) hide)
     )
@@
       (effects (font (size 1.27 1.27)) hide)
     )
+    (property "Config" "-SR" (id 6) (at 134.62 111.76 0)
+      (effects (font (size 1.27 1.27)) hide)
+    )
     (pin "1")
     (pin "2")
@@
       (effects (font (size 1.27 1.27)) hide)
     )
+    (property "Config" "-SR" (id 6) (at 119.38 132.08 0)
+      (effects (font (size 1.27 1.27)) hide)
+    )
     (pin "1")
     (pin "2")
@@
       (effects (font (size 1.27 1.27)) hide)
     )
+    (property "Config" "-SR" (id 6) (at 140.97 57.15 0)
+      (effects (font (size 1.27 1.27)) hide)
+    )
