File: PCB/mobo/Mosfets.kicad_sch (KiCad schematic)
At the start: 4 parts, among them U4 CSD88537ND, U5 CSD88537ND, U6 CSD88537ND

Commit message: Pretty stable naming and xlsx output
Parts:
- R11: Config (none) -> -GR
Changed lines of the file:
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@@
+      (effects (font (size 1.27 1.27)) hide)
+    )
+    (property "Config" "-GR" (id 6) (at 151.13 115.57 0)
       (effects (font (size 1.27 1.27)) hide)
     )
